File: Hardware/MAX3232_Breakout.brd (EAGLE design)
At the start: 25.4 x 14 mm, 12 parts, among them U1 MAX3232

Commit message: switched fids to regular size
Parts:
- removed JP3, JP4: FIDUCIALUFIDUCIAL, SparkFun:MICRO-FIDUCIAL
- added FID1, FID2: FIDUCIAL1X2, SparkFun-Aesthetics:FIDUCIAL-1X2
