File: Hardware/MAX3232_Breakout.sch (EAGLE design)
At the start: 12 parts, among them U1 MAX3232

Commit message: switched fids to regular size
Parts:
- removed JP3, JP4: FIDUCIALUFIDUCIAL, SparkFun:FIDUCIALUFIDUCIAL
- added FID1, FID2: FIDUCIAL1X2, SparkFun-Aesthetics:FIDUCIAL1X2
Changed lines of the file:
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@@
 <?xml version="1.0" encoding="utf-8"?>
 <!DOCTYPE eagle SYSTEM "eagle.dtd">
-<eagle version="6.4">
+<eagle version="6.6.0">
 <drawing>
 <settings>
@@
 <attribute name="SPARKLE_ID" value="918"/>
 </part>
-<part name="JP3" library="SparkFun" deviceset="FIDUCIAL" device="UFIDUCIAL"/>
-<part name="JP4" library="SparkFun" deviceset="FIDUCIAL" device="UFIDUCIAL"/>
 <part name="LOGO1" library="SparkFun-Aesthetics" deviceset="SFE_LOGO_FLAME" device=".1_INCH"/>
 <part name="P+2" library="SparkFun-Aesthetics" deviceset="VCC" device=""/>
 <part name="GND3" library="SparkFun-Aesthetics" deviceset="GND" device=""/>
+<part name="FID1" library="SparkFun-Aesthetics" deviceset="FIDUCIAL" device="1X2"/>
+<part name="FID2" library="SparkFun-Aesthetics" deviceset="FIDUCIAL" device="1X2"/>
 </parts>
 <sheets>
@@
 <attribute name="VALUE" x="178.054" y="121.793" size="1.778" layer="96" rot="R180"/>
 </instance>
-<instance part="JP3" gate="G$1" x="223.52" y="33.02"/>
-<instance part="JP4" gate="G$1" x="223.52" y="27.94"/>
 <instance part="LOGO1" gate="G$1" x="213.36" y="38.1"/>
 <instance part="P+2" gate="1" x="45.72" y="104.14"/>
 <instance part="GND3" gate="1" x="45.72" y="93.98"/>
+<instance part="FID1" gate="G$1" x="226.06" y="20.32"/>
+<instance part="FID2" gate="G$1" x="231.14" y="20.32"/>
 </instances>
 <busses>
